File: keypad_pcb/merch-hat.brd (EAGLE design)
At the start: 65 x 56 mm, 15 parts

Commit message: update pcbs to remove clear bug on 74174 chip
Connections:
- net +5V: now also SELECT_BITS.1
- net GND: no longer SELECT_BITS.1
Routing:
- net GND: track 116.0 -> 101.2 mm
Changed lines of the file:
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@@
 <?xml version="1.0" encoding="utf-8"?>
 <!DOCTYPE eagle SYSTEM "eagle.dtd">
-<eagle version="7.6.0">
+<eagle version="8.0.1">
 <drawing>
 <settings>
@@
 <contactref element="ROW_MUX" pad="7"/>
 <contactref element="SELECT_BITS" pad="14"/>
-<contactref element="SELECT_BITS" pad="1"/>
 <contactref element="COL_DEMUX" pad="2"/>
 <contactref element="COL_DEMUX" pad="1"/>
@@
 <wire x1="11.938" y1="13.208" x2="25.146" y2="13.208" width="0.4064" layer="1"/>
 <wire x1="25.146" y1="13.208" x2="26.416" y2="14.478" width="0.4064" layer="1"/>
-<wire x1="41.91" y1="40.894" x2="39.37" y2="40.894" width="0.4064" layer="1"/>
 <wire x1="41.91" y1="40.894" x2="46.99" y2="35.814" width="0.4064" layer="1"/>
 <wire x1="36.322" y1="23.114" x2="34.036" y2="20.828" width="0.4064" layer="1"/>
@@
 <wire x1="28.702" y1="20.828" x2="26.416" y2="23.114" width="0.4064" layer="1"/>
 <wire x1="36.322" y1="23.114" x2="39.37" y2="23.114" width="0.4064" layer="1"/>
-<wire x1="39.37" y1="40.894" x2="41.91" y2="38.354" width="0.4064" layer="1"/>
 <wire x1="41.91" y1="38.354" x2="41.91" y2="25.654" width="0.4064" layer="1"/>
 <wire x1="41.91" y1="25.654" x2="39.37" y2="23.114" width="0.4064" layer="1"/>
-<wire x1="33.274" y1="46.99" x2="39.37" y2="40.894" width="0.4064" layer="16"/>
 <wire x1="33.147" y1="47.117" x2="32.004" y2="48.26" width="0.4064" layer="16"/>
 <wire x1="32.004" y1="48.26" x2="21.5" y2="48.26" width="0.4064" layer="16"/>
@@
 <wire x1="27.686" y1="19.558" x2="27.686" y2="15.748" width="0.4064" layer="1"/>
 <wire x1="27.686" y1="15.748" x2="26.416" y2="14.478" width="0.4064" layer="1"/>
+<wire x1="41.91" y1="38.354" x2="41.91" y2="40.894" width="0" layer="19" extent="1-1"/>
+<wire x1="43.942" y1="46.99" x2="41.91" y2="40.894" width="0" layer="19" extent="1-1"/>
 </signal>
 <signal name="+5V">
@@
 <wire x1="26.67" y1="48.26" x2="39.624" y2="48.26" width="0.4064" layer="1"/>
 <wire x1="39.624" y1="48.26" x2="46.99" y2="40.894" width="0.4064" layer="1"/>
+<contactref element="SELECT_BITS" pad="1"/>
+<wire x1="36.576" y1="39.624" x2="39.37" y2="40.894" width="0" layer="19" extent="1-1"/>
 </signal>
 <signal name="N$2">
